File: loadcell_4way.kicad_pcb (KiCad board)
At the start: 2 copper layers, 60 x 40 mm, 76 parts, among them J1 USB_B_Micro, J2 Battery, J3 OLDED_Screen, J4 Load Cell, Q1 FDS6892A, Q2 BSS138, Q3 SM2331PSA P-MOSFET, Q4 S8550, Q5 BSS138, SW1 SW_Push, SW2 SW_Push, SW3 SW_Push, U1 FS312F-G, U2 MT3608, U3 TP4056, U4 CH330N, U5 LM1117-3.3, U7 HX711

Commit message: wip
Parts:
- removed C11: 100nF, Capacitor_SMD:C_0603_1608Metric
- removed Q4: S8550, Package_TO_SOT_SMD:SOT-23
- removed R24: 100k, Resistor_SMD:R_0603_1608Metric
- removed R25: 10k, Resistor_SMD:R_0603_1608Metric
- removed R27: 0R, Resistor_SMD:R_0603_1608Metric
- removed U7: HX711, Package_SO:SOP-16_4.55x10.3mm_P1.27mm
- added C17: 100nF, Capacitor_SMD:C_0603_1608Metric, F.Cu at (119.6, 80.9)
- added C18: 100nF, Capacitor_SMD:C_0603_1608Metric, F.Cu at (227.2, 86.6)
- added C19: 100nF, Capacitor_SMD:C_0603_1608Metric, F.Cu at (227.2, 82.7)
- added C21: 100nF, Capacitor_SMD:C_0603_1608Metric, F.Cu at (165.2, 50.2)
- added C22: 100nF, Capacitor_SMD:C_0603_1608Metric, F.Cu at (188.0, 67.8)
- added C23: 10uF, Capacitor_SMD:C_0603_1608Metric, F.Cu at (165.2, 51.9)
- added C24: 10uF, Capacitor_SMD:C_0603_1608Metric, F.Cu at (184.4, 76.5)
- added C25: 10uF, Capacitor_SMD:C_0603_1608Metric, F.Cu at (184.4, 73.3)
- added C26: 100nF, Capacitor_SMD:C_0603_1608Metric, F.Cu at (182.8, 73.3)
- added C27: 100nF, Capacitor_SMD:C_0603_1608Metric, F.Cu at (166.4, 74.1)
- added C28: 100nF, Capacitor_SMD:C_0603_1608Metric, F.Cu at (166.6, 69.1)
- added C29: 100nF, Capacitor_SMD:C_0603_1608Metric, F.Cu at (178.5, 74.0)
- added C30: 100nF, Capacitor_SMD:C_0603_1608Metric, F.Cu at (178.5, 71.8)
- added J5: T4145015051-001, Loadcell:TE_T4145015051-001, F.Cu at (153.3, 90.5)
- added J6: T4145015051-001, Loadcell:TE_T4145015051-001, F.Cu at (186.7, 90.5)
- added J7: T4145015051-001, Loadcell:TE_T4145015051-001, F.Cu at (220.0, 90.5)
- added Q7: BSS138, Package_TO_SOT_SMD:SOT-23, F.Cu at (115.3, 75.6)
- added Q8: BSS138, Package_TO_SOT_SMD:SOT-23, F.Cu at (119.1, 75.6)
- added R17: 1k, Resistor_SMD:R_0603_1608Metric, F.Cu at (156.1, 82.7)
- added R29: 1k, Resistor_SMD:R_0603_1608Metric, F.Cu at (122.0, 81.8)
- added R30: 1k, Resistor_SMD:R_0603_1608Metric, F.Cu at (224.9, 83.6)
- added R31: 10k, Resistor_SMD:R_0603_1608Metric, F.Cu at (165.2, 53.5)
- added R32: 10k, Resistor_SMD:R_0603_1608Metric, F.Cu at (178.2, 66.0)
- added R33: 10k, Resistor_SMD:R_0603_1608Metric, F.Cu at (189.0, 51.0)
- added R34: 10k, Resistor_SMD:R_0603_1608Metric, F.Cu at (116.3, 71.4)
- added R35: 10k, Resistor_SMD:R_0603_1608Metric, F.Cu at (118.1, 71.4)
- added R36: 390k, Resistor_SMD:R_0603_1608Metric, F.Cu at (189.6, 67.8)
- added R37: 100k, Resistor_SMD:R_0603_1608Metric, F.Cu at (186.4, 67.8)
- added R38: 10k, Resistor_SMD:R_0603_1608Metric, F.Cu at (178.5, 70.2)
- added U10: ADS1234IPW, Loadcell:SOP65P640X120-28N, F.Cu at (172.4, 72.8)
- added U11: LM1117-3.3, Package_TO_SOT_SMD:SOT-223, F.Cu at (189.8, 75.4)
- added U9: CH340C, Package_SO:SOIC-16_3.9x9.9mm_P1.27mm, F.Cu at (116.0, 65.0)
- C12, C15: value 10uF -> 100nF
- H1, H2, H3, H4: value MountingHole -> PCB Mounting hole; footprint forcegauge:MountingHole_2mm_OLED -> MountingHole:MountingHole_3.2mm_M3
- H5, H6, H7, H8: value PCB Mounting hole -> MountingHole; footprint forcegauge:MountingHole_2mm_OLED -> Loadcell:MountingHole_2mm_OLED
- J2: footprint Connector_PinHeader_2.54mm:PinHeader_1x02_P2.54mm_Vertical -> Connector_JST:JST_PH_B2B-PH-SM4-TB_1x02-1MP_P2.00mm_Vertical
- J4: value Load Cell -> T4145015051-001; footprint Connector_PinSocket_2.54mm:PinSocket_1x05_P2.54mm_Vertical -> Loadcell:TE_T4145015051-001
- R1: value 100 -> 2k
- R10: value 1k -> 470R
- R12: value 470R -> 100
- R13: value 100k -> 0R
- R14, R16: value 10k -> 4k7
- R15: value 100 -> 100k
- R18, R26, R28: value 10k -> 1k
- R19: value 0R -> 1k
- R20: value 20k -> 1k
- R21: value 8k2 -> 10k
- R22, R5: value 1k -> 100
- R23: value 1k -> 100k
- R3: value 2k -> 7.5k
- R4: value 7.5k -> 1k
- R6: value 100 -> 1k
- R7: value 1k -> 390k
- R8: value 390k -> 100k
- R9: value 100k -> 1k
- U3: footprint forcegauge:SOP8-PP -> Loadcell:SOP8-PP
- U4: value CH330N -> ESP32-C3-WROOM-02; footprint Package_SO:SOIC-8_3.9x4.9mm_P1.27mm -> Loadcell:ESP32-C3-WROOM-02
- moved R26 107.5 mm to (229.5, 83.7), turned to 90 degrees
- moved R14 106.5 mm to (224.0, 66.0)
- moved BZ1 101.0 mm to (208.0, 51.8), turned to 90 degrees
- moved R12 84.9 mm to (197.9, 44.4)
- moved R16 83.8 mm to (224.0, 69.0), turned to 0 degrees
- moved H5 83.3 mm to (197.5, 81.0)
- moved Q2 82.6 mm to (197.9, 47.9), turned to -90 degrees
- moved H4 81.1 mm to (235.0, 45.0), turned to 0 degrees
- moved H7 80.1 mm to (197.5, 59.0)
- moved J2 78.5 mm to (115.0, 45.0), turned to 0 degrees
- moved C5 70.5 mm to (123.1, 45.4)
- moved R8 70.4 mm to (188.0, 64.6), turned to 90 degrees
- moved H3 70.2 mm to (105.0, 45.0), turned to 0 degrees
- moved C8 69.5 mm to (186.4, 64.6), turned to 90 degrees
- moved U1 66.2 mm to (123.3, 48.3), turned to 90 degrees
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Connections:
- BZ1 pad 2: (no net) -> Net-(BZ1-+)
- C12 pad 1: E- -> +3.3VA
- C12 pad 2: E+ -> Net-(C12-Pad2)
- C13 pad 1: (no net) -> +3.3VA
- C13 pad 2: E- -> Net-(C13-Pad2)
- C14 pad 1: (no net) -> A2+
- C14 pad 2: (no net) -> A2-
- C15 pad 1: GND -> +3.3VA
- C15 pad 2: +5V -> Net-(C15-Pad2)
- C16 pad 1: +3V3 -> A3+
- C16 pad 2: GND -> A3-
- C4 pad 1: (no net) -> +3V3
- C5 pad 1: (no net) -> Net-(U1-VCC)
- C8 pad 1: V_BAT -> VBAT_FB
- D1 pad 2: (no net) -> Net-(D1-A)
- D2 pad 1: (no net) -> Net-(D2-K)
- D2 pad 2: (no net) -> Net-(D2-A)
- D3 pad 1: (no net) -> Net-(D3-K)
- D3 pad 2: (no net) -> Net-(D3-A)
- D4 pad 1: (no net) -> Net-(D4-K)
- D4 pad 2: BTN_2 -> Net-(D4-A)
- D5 pad 1: (no net) -> Net-(D4-K)
- D5 pad 2: (no net) -> BTN_2
- J1 pad 4: (no net) -> unconnected-(J1-ID-Pad4)
- J3 pad 3: SCL -> ESP32_IO9
- J4 pad 1: E+ -> +3.3VA
- J4 pad 2: E- -> Net-(C12-Pad2)
- J4 pad 3: A- -> Net-(J4-Pad3)
- J4 pad 4: A+ -> Net-(J4-Pad4)
- L1 pad 2: (no net) -> Net-(D1-A)
- Q1 pad 2: (no net) -> Net-(Q1A-G1)
- Q1 pad 4: (no net) -> Net-(Q1B-G2)
- Q1 pad 5: (no net) -> Net-(Q1A-D1-Pad7)
- Q1 pad 6: (no net) -> Net-(Q1A-D1-Pad7)
- Q1 pad 7: (no net) -> Net-(Q1A-D1-Pad7)
- Q1 pad 8: (no net) -> Net-(Q1A-D1-Pad7)
- Q2 pad 1: (no net) -> Net-(Q2-G)
- Q2 pad 3: (no net) -> Net-(BZ1-+)
- Q3 pad 1: (no net) -> Net-(D4-A)
- Q5 pad 1: (no net) -> Net-(Q5-G)
- Q5 pad 3: (no net) -> Net-(D4-A)
- R1 pad 1: (no net) -> Net-(U1-CS)
- R1 pad 2: BUZZER -> BAT-
- R10 pad 1: (no net) -> Net-(U9-TXD)
- R10 pad 2: VBUS -> RXD
- R11 pad 1: (no net) -> Net-(U9-RXD)
- R11 pad 2: RXD -> TXD
- R12 pad 1: (no net) -> Net-(Q2-G)
- R12 pad 2: TXD -> BUZZER
- R13 pad 1: (no net) -> GNDA
- R13 pad 2: BAT+ -> GND
- R14 pad 1: +3V3 -> SDA
- R14 pad 2: (no net) -> +3V3
- R15 pad 1: PWR_EN -> Net-(D4-A)
- R15 pad 2: (no net) -> BAT+
- R16 pad 1: +3V3 -> ESP32_IO9
- R16 pad 2: BTN_1 -> +3V3
- R18 pad 1: +3V3 -> Net-(J5-Pad4)
- R18 pad 2: (no net) -> A2-
- R19 pad 1: E- -> Net-(J6-Pad3)
- R19 pad 2: GND -> A3+
- R2 pad 1: (no net) -> Net-(U3-PROG)
- R2 pad 2: BAT- -> GND
- R20 pad 1: E+ -> Net-(J6-Pad4)
- R20 pad 2: (no net) -> A3-
- R21 pad 1: (no net) -> GND
- R21 pad 2: E- -> Net-(Q5-G)
- R22 pad 1: A- -> PWR_EN
- R22 pad 2: (no net) -> Net-(Q5-G)
- R23 pad 1: A+ -> BTN_2
- R23 pad 2: (no net) -> +3V3
- R26 pad 1: GND -> Net-(J7-Pad3)
- R26 pad 2: BUZZER -> A4+
- R28 pad 1: GND -> Net-(J4-Pad4)
- R28 pad 2: (no net) -> A1-
- R3 pad 1: (no net) -> Net-(U2-FB)
- R3 pad 2: GND -> +5V
- R4 pad 1: (no net) -> GND
- R4 pad 2: +5V -> Net-(U2-FB)
- R5 pad 1: GND -> BAT+
- R5 pad 2: (no net) -> Net-(U1-VCC)
- R6 pad 1: BAT+ -> Net-(D2-A)
- R6 pad 2: (no net) -> VBUS
- R7 pad 1: (no net) -> VCC
- R7 pad 2: VBUS -> VBAT_FB
- R8 pad 1: VCC -> VBAT_FB
- R8 pad 2: V_BAT -> GND
- R9 pad 1: V_BAT -> Net-(D3-A)
- R9 pad 2: GND -> VBUS
- SW2 pad 1: (no net) -> BTN_3
- SW3 pad 1: BTN_3 -> Net-(D4-K)
- U1 pad 1: (no net) -> Net-(Q1B-G2)
- U1 pad 2: (no net) -> Net-(U1-CS)
- U1 pad 3: (no net) -> Net-(Q1A-G1)
- U1 pad 4: (no net) -> unconnected-(U1-TD-Pad4)
- U1 pad 5: (no net) -> Net-(U1-VCC)
- U2 pad 1: (no net) -> Net-(D1-A)
- U2 pad 3: (no net) -> Net-(U2-FB)
- U2 pad 6: (no net) -> unconnected-(U2-NC-Pad6)
- U3 pad 2: (no net) -> Net-(U3-PROG)
- U3 pad 6: (no net) -> Net-(D3-K)
- U3 pad 7: (no net) -> Net-(D2-K)
- U4 pad 1: D+ -> +3V3
- U4 pad 2: D- -> ESP32_EN
- U4 pad 3: GND -> MUX0
- U4 pad 4: (no net) -> MUX1
- U4 pad 5: +3V3 -> CLK
- U4 pad 6: (no net) -> DOUT
- U4 pad 7: (no net) -> SDA
- U4 pad 8: (no net) -> ESP32_IO9
Routing:
- net (no net): track 182.0 -> 0.00 mm, vias 10 -> 0
- net +3V3: track 121.1 -> 0.00 mm, vias 4 -> 0
- net +5V: track 85.7 -> 0.00 mm, vias 2 -> 0
- net VCC: track 76.5 -> 0.00 mm, vias 2 -> 0
- net VBUS: track 52.7 -> 0.00 mm, vias 3 -> 0
- net SDA: track 49.9 -> 0.00 mm
- net SCL: track 48.5 -> 0.00 mm
- net CLK: track 42.5 -> 0.00 mm
- net BTN_2: track 40.5 -> 0.00 mm
- net PWR_EN: track 38.0 -> 0.00 mm, vias 1 -> 0
- net BAT+: track 34.8 -> 0.00 mm
- net DOUT: track 33.7 -> 0.00 mm, vias 2 -> 0
- net BAT-: track 30.9 -> 0.00 mm, vias 1 -> 0
- net TXD: track 29.3 -> 0.00 mm, vias 1 -> 0
- net BTN_3: track 24.3 -> 0.00 mm, vias 1 -> 0
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Other:
- board size 60 x 40 mm -> 140 x 60 mm
- board text removed: "Forcegauge© v0.4"
- board text removed: "by Beni"

Commit message: pcb
Parts:
- moved J2 6.75 mm to (115.0, 51.8)
Other:
- outline, holes or cut-outs redrawn
Changed lines of the file:
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@@
   )
   (footprint "Connector_JST:JST_PH_B2B-PH-SM4-TB_1x02-1MP_P2.00mm_Vertical" (layer "F.Cu")
-    (at 115 45)
+    (at 115 51.75)
     (descr "JST PH series connector, B2B-PH-SM4-TB (http://www.jst-mfg.com/product/pdf/eng/ePH.pdf), generated with kicad-footprint-generator")
     (tags "connector JST PH side entry")
@@
     )
   )
-  (gr_rect (start 100 40) (end 240 100)
-    (stroke (width 0.1) (type default)) (fill none) (layer "Edge.Cuts"))
+  (gr_line (start 100 40) (end 100 100)
+    (stroke (width 0.1) (type default)) (layer "Edge.Cuts"))
+  (gr_line (start 110 40) (end 100 40)
+    (stroke (width 0.1) (type default)) (layer "Edge.Cuts"))
+  (gr_line (start 100 100) (end 240 100)
+    (stroke (width 0.1) (type default)) (layer "Edge.Cuts"))
+  (gr_line (start 240 100) (end 240 40)
+    (stroke (width 0.1) (type default)) (layer "Edge.Cuts"))
+  (gr_line (start 112 43) (end 118 43)
+    (stroke (width 0.1) (type default)) (layer "Edge.Cuts"))
+  (gr_line (start 240 40) (end 120 40)
+    (stroke (width 0.1) (type default)) (layer "Edge.Cuts"))
+  (gr_line (start 118 43) (end 120 40)
+    (stroke (width 0.1) (type default)) (layer "Edge.Cuts"))
+  (gr_line (start 110 40) (end 112 43)
+    (stroke (width 0.1) (type default)) (layer "Edge.Cuts"))
   (gr_text "B-" (at 170.18 106.95) (layer "F.SilkS")
     (effects (font (size 0.8128 0.8128) (thickness 0.1524)))

Commit message: wip
Parts:
- removed J7: T4145015051-001, Loadcell:TE_T4145015051-001
- removed U11: LM1117-3.3, Package_TO_SOT_SMD:SOT-223
- added J10: Conn_01x05, Connector_Phoenix_MSTB:PhoenixContact_MSTBA_2,5_5-G-5,08_1x05_P5.08mm_Horizontal, F.Cu at (113.0, 96.0)
- added R24: 10k, Resistor_SMD:R_0603_1608Metric, F.Cu at (174.5, 83.5)
- added R25: 2k2, Resistor_SMD:R_0603_1608Metric, F.Cu at (177.0, 83.5)
- added U7: AP2127K-ADJ, Package_TO_SOT_SMD:SOT-23-5, F.Cu at (171.0, 83.0)
- J4, J5, J6: value T4145015051-001 -> Conn_01x05; footprint Loadcell:TE_T4145015051-001 -> Connector_Phoenix_MSTB:PhoenixContact_MSTBA_2,5_5-G-5,08_1x05_P5.08mm_Horizontal
- moved J4 24.9 mm to (144.3, 96.0)
- moved J5 22.9 mm to (175.6, 96.0)
- moved J6 20.9 mm to (206.8, 96.0)
Connections:
- C12 pad 2: Net-(C12-Pad2) -> Net-(J10-Pin_2)
- C13 pad 2: Net-(C13-Pad2) -> Net-(J4-Pin_2)
- C15 pad 2: Net-(C15-Pad2) -> Net-(J5-Pin_2)
- C18 pad 2: Net-(C18-Pad2) -> Net-(J6-Pin_2)
- J4 pad 2: Net-(C12-Pad2) -> Net-(J4-Pin_2)
- J4 pad 3: Net-(J4-Pad3) -> Net-(J4-Pin_3)
- J4 pad 4: Net-(J4-Pad4) -> Net-(J4-Pin_4)
- J5 pad 2: Net-(C13-Pad2) -> Net-(J5-Pin_2)
- J5 pad 3: Net-(J5-Pad3) -> Net-(J5-Pin_3)
- J5 pad 4: Net-(J5-Pad4) -> Net-(J5-Pin_4)
- J6 pad 2: Net-(C15-Pad2) -> Net-(J6-Pin_2)
- J6 pad 3: Net-(J6-Pad3) -> Net-(J6-Pin_3)
- J6 pad 4: Net-(J6-Pad4) -> Net-(J6-Pin_4)
- R17 pad 1: Net-(J5-Pad3) -> Net-(J4-Pin_3)
- R18 pad 1: Net-(J5-Pad4) -> Net-(J4-Pin_4)
- R19 pad 1: Net-(J6-Pad3) -> Net-(J5-Pin_3)
- R20 pad 1: Net-(J6-Pad4) -> Net-(J5-Pin_4)
- R26 pad 1: Net-(J7-Pad3) -> Net-(J6-Pin_3)
- R28 pad 1: Net-(J4-Pad4) -> Net-(J10-Pin_4)
- R29 pad 1: Net-(J4-Pad3) -> Net-(J10-Pin_3)
- R30 pad 1: Net-(J7-Pad4) -> Net-(J6-Pin_4)

Commit message: wip
Parts:
- added C11: 100nF, Capacitor_SMD:C_0603_1608Metric, F.Cu at (128.0, 85.0)
- added C20: 100nF, Capacitor_SMD:C_0603_1608Metric, F.Cu at (123.0, 85.0)
- added C31: 100nF, Capacitor_SMD:C_0603_1608Metric, F.Cu at (160.0, 85.0)
- added C32: 100nF, Capacitor_SMD:C_0603_1608Metric, F.Cu at (155.0, 85.0)
- added C33: 100nF, Capacitor_SMD:C_0603_1608Metric, F.Cu at (191.0, 85.0)
- added C34: 100nF, Capacitor_SMD:C_0603_1608Metric, F.Cu at (185.8, 85.0)
- added C35: 100nF, Capacitor_SMD:C_0603_1608Metric, F.Cu at (222.0, 85.0)
- added C36: 100nF, Capacitor_SMD:C_0603_1608Metric, F.Cu at (217.0, 85.0)
- added C37: 100nF, Capacitor_SMD:C_0603_1608Metric, F.Cu at (172.3, 85.3)
- added C38: 100nF, Capacitor_SMD:C_0603_1608Metric, F.Cu at (167.2, 81.1)
- added FB1: FerriteBead, Inductor_SMD:L_1206_3216Metric, F.Cu at (168.2, 83.3)
- moved C18 17.8 mm to (210.0, 91.0)
- moved C24 16.2 mm to (172.2, 87.1), turned to 0 degrees
- moved C15 14.9 mm to (178.0, 91.0)
- moved R26 14.0 mm to (217.0, 90.0)
- moved R28 13.6 mm to (128.0, 90.0)
- moved R19 11.0 mm to (186.0, 90.0)
- moved R18 10.7 mm to (159.0, 90.0)
- moved C17 8.68 mm to (125.8, 87.0), turned to 0 degrees
- moved C19 8.58 mm to (219.8, 87.0), turned to 0 degrees
- moved C13 8.30 mm to (147.0, 91.0)
- moved R29 8.26 mm to (123.0, 90.0)
- moved R17 7.62 mm to (154.0, 90.0)
- moved R20 7.30 mm to (191.0, 90.0)
- moved R30 7.03 mm to (222.0, 90.0)
- moved C14 6.18 mm to (157.0, 87.0), turned to 0 degrees
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Connections:
- C12 pad 1: +3.3VA -> VDDA
- C13 pad 1: +3.3VA -> VDDA
- C15 pad 1: +3.3VA -> VDDA
- C18 pad 1: +3.3VA -> VDDA
- C24 pad 1: +5V -> Net-(U7-EN)
- C25 pad 1: +3.3VA -> VDDA
- C26 pad 1: +3.3VA -> VDDA
- C29 pad 1: +3.3VA -> VDDA
- J10 pad 1: +3.3VA -> VDDA
- J4 pad 1: +3.3VA -> VDDA
- J5 pad 1: +3.3VA -> VDDA
- J6 pad 1: +3.3VA -> VDDA
- R24 pad 2: +3.3VA -> VDDA
- U10 pad 22: +3.3VA -> VDDA
- U7 pad 1: +5V -> Net-(U7-EN)
- U7 pad 3: +5V -> Net-(U7-EN)
- U7 pad 5: +3.3VA -> VDDA

Commit message: pcb wip
Parts:
- moved R36 66.6 mm to (123.7, 58.1)
- moved C22 64.6 mm to (123.7, 61.4), turned to -90 degrees
- moved R37 61.3 mm to (125.4, 61.4), turned to -90 degrees
- moved R22 44.3 mm to (189.6, 54.0), turned to 0 degrees
- moved R23 43.4 mm to (189.6, 55.6), turned to 0 degrees
- moved D2 40.7 mm to (110.4, 61.0)
- moved D3 40.7 mm to (110.4, 59.4)
- moved R2 40.7 mm to (122.0, 61.4)
- moved R6 40.7 mm to (110.4, 62.6)
- moved R9 40.7 mm to (110.4, 64.3)
- moved U3 40.7 mm to (116.4, 60.0)
- moved R21 37.9 mm to (137.6, 42.4)
- moved R15 36.4 mm to (131.0, 46.6), turned to -90 degrees
- moved Q5 35.9 mm to (133.9, 43.6), turned to 0 degrees
- moved Q3 32.0 mm to (133.9, 47.2), turned to 0 degrees
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
Commit message: PCB wip
Parts:
- added C39: 100nF, Capacitor_SMD:C_0603_1608Metric, F.Cu at (172.2, 66.8)
- added R27: 0R, Resistor_SMD:R_0603_1608Metric, F.Cu at (106.2, 89.2)
- added R39: 0R, Resistor_SMD:R_0603_1608Metric, F.Cu at (106.2, 87.4)
- moved R13 73.6 mm to (111.6, 88.5)
- moved R33 64.0 mm to (128.8, 70.9), turned to -90 degrees
- moved R7 50.0 mm to (141.6, 50.7)
- moved R8 50.0 mm to (140.0, 50.7)
- moved C8 45.4 mm to (143.2, 50.7)
- moved R32 35.4 mm to (144.3, 55.8), turned to 90 degrees
- moved C26 20.4 mm to (160.1, 68.7), turned to -90 degrees
- moved C25 17.9 mm to (161.7, 68.7), turned to -90 degrees
- moved C4 10.7 mm to (120.5, 74.5)
- moved C2 10.7 mm to (122.1, 74.5)
- moved C3 10.5 mm to (123.7, 74.5)
- moved C38 10.4 mm to (150.5, 74.1), turned to 90 degrees
- moved BZ1 7.60 mm to (210.1, 44.5), turned to -90 degrees
- moved FB1 7.21 mm to (152.6, 73.2), turned to 90 degrees
- moved C24 5.19 mm to (155.7, 75.0)
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Connections:
- C12 pad 2: Net-(J10-Pin_2) -> GNDA
- C13 pad 2: Net-(J4-Pin_2) -> GNDA
- C15 pad 2: Net-(J5-Pin_2) -> GNDA
- C18 pad 2: Net-(J6-Pin_2) -> GNDA
- C30 pad 1: +3.3VA -> VDDA
- J10 pad 2: Net-(J10-Pin_2) -> GNDA
- J10 pad 5: GND -> Earth
- J4 pad 2: Net-(J4-Pin_2) -> GNDA
- J4 pad 5: GND -> Earth
- J5 pad 2: Net-(J5-Pin_2) -> GNDA
- J5 pad 5: GND -> Earth
- J6 pad 2: Net-(J6-Pin_2) -> GNDA
- J6 pad 5: GND -> Earth
- U10 pad 13: A3+ -> A2+
- U10 pad 14: A3- -> A2-
- U10 pad 15: A4- -> A3-
- U10 pad 16: A4+ -> A3+
- U10 pad 17: A2- -> A4-
- U10 pad 18: A2+ -> A4+
- U10 pad 20: +3.3VA -> VDDA
Routing:
- net VDDA: track 0.00 -> 290.4 mm, vias 0 -> 8
- net +3V3: track 0.00 -> 228.0 mm, vias 0 -> 8
- net Earth: track 0.00 -> 145.3 mm, vias 0 -> 2
- net ESP32_IO9: track 0.00 -> 143.3 mm, vias 0 -> 3
- net +5V: track 0.00 -> 115.7 mm, vias 0 -> 8
- net Net-(D4-K): track 0.00 -> 90.7 mm, vias 0 -> 1
- net ESP32_EN: track 0.00 -> 84.3 mm, vias 0 -> 2
- net BTN_3: track 0.00 -> 78.9 mm, vias 0 -> 3
- net TXD: track 0.00 -> 74.0 mm
- net RXD: track 0.00 -> 72.2 mm
- net VBUS_FB: track 0.00 -> 69.2 mm, vias 0 -> 2
- net BTN_2: track 0.00 -> 67.7 mm, vias 0 -> 2
- net Net-(Q5-G): track 0.00 -> 64.9 mm, vias 0 -> 2
- net SDA: track 0.00 -> 60.9 mm, vias 0 -> 1
- net VBAT_FB: track 0.00 -> 60.8 mm, vias 0 -> 2
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- added copper zone on B.Cu, net GND
- added copper zone on F.Cu, net GND
- added copper zone on B.Cu, net GNDA
- added copper zone on F.Cu, net GNDA

Commit message: pcb wip
Parts:
- removed J10: Conn_01x05, Connector_Phoenix_MSTB:PhoenixContact_MSTBA_2,5_5-G-5,08_1x05_P5.08mm_Horizontal
- added J7: T4145015051-001, Loadcell:TE_T4145015051-001, F.Cu at (214.0, 90.8)
- J4, J5, J6: value Conn_01x05 -> T4145015051-001; footprint Connector_Phoenix_MSTB:PhoenixContact_MSTBA_2,5_5-G-5,08_1x05_P5.08mm_Horizontal -> Loadcell:TE_T4145015051-001
- moved J6 22.8 mm to (184.7, 90.8)
- moved J5 20.9 mm to (155.3, 90.8)
- moved J4 19.0 mm to (126.0, 90.8)
- moved C12 10.7 mm to (126.0, 86.6)
- moved C13 9.00 mm to (154.8, 86.5)
- moved C15 8.09 mm to (184.7, 86.5)
- moved R28 6.86 mm to (125.8, 83.5), turned to 0 degrees
- moved R18 6.71 mm to (157.0, 83.6), turned to 0 degrees
- moved R20 6.49 mm to (187.5, 84.5), turned to 90 degrees
- moved R29 6.40 mm to (127.0, 85.0), turned to 180 degrees
- moved R30 6.03 mm to (218.5, 85.8), turned to 90 degrees
- moved R17 5.87 mm to (158.0, 85.7), turned to 180 degrees
- moved C18 5.84 mm to (213.7, 86.5)
- moved BZ1 5.00 mm to (210.1, 39.5)
- moved C1 5.00 mm to (146.5, 40.6)
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Connections:
- net Earth renamed SHIELD
- J4 pad 3: Net-(J4-Pin_3) -> Net-(J4-Pad3)
- J4 pad 4: Net-(J4-Pin_4) -> Net-(J4-Pad4)
- J5 pad 3: Net-(J5-Pin_3) -> Net-(J5-Pad3)
- J5 pad 4: Net-(J5-Pin_4) -> Net-(J5-Pad4)
- J6 pad 3: Net-(J6-Pin_3) -> Net-(J6-Pad3)
- J6 pad 4: Net-(J6-Pin_4) -> Net-(J6-Pad4)
- R17 pad 1: Net-(J4-Pin_3) -> Net-(J5-Pad3)
- R18 pad 1: Net-(J4-Pin_4) -> Net-(J5-Pad4)
- R19 pad 1: Net-(J5-Pin_3) -> Net-(J6-Pad3)
- R20 pad 1: Net-(J5-Pin_4) -> Net-(J6-Pad4)
- R26 pad 1: Net-(J6-Pin_3) -> Net-(J7-Pad3)
- R28 pad 1: Net-(J10-Pin_4) -> Net-(J4-Pad4)
- R29 pad 1: Net-(J10-Pin_3) -> Net-(J4-Pad3)
- R30 pad 1: Net-(J6-Pin_4) -> Net-(J7-Pad4)
Routing:
- net VDDA: track 290.4 -> 180.0 mm, vias 8 -> 4
- net Net-(J7-Pad4): track 0.00 -> 16.0 mm
- net Net-(J6-Pad4): track 0.00 -> 13.5 mm
- net Net-(J5-Pad4): track 0.00 -> 13.1 mm
- net GND: track 33.9 -> 46.7 mm, vias 96 -> 102
- net Net-(J4-Pad4): track 0.00 -> 10.8 mm
- net Net-(J4-Pad3): track 0.00 -> 9.18 mm
- net Net-(J5-Pin_3): track 8.79 -> 0.00 mm
- net Net-(J6-Pad3): track 0.00 -> 8.46 mm
- net Net-(J7-Pad3): track 0.00 -> 7.63 mm
- net Net-(J5-Pad3): track 0.00 -> 7.53 mm
- net Net-(D4-K): track 90.7 -> 97.6 mm
- net Net-(J6-Pin_3): track 6.55 -> 0.00 mm
- net Net-(J6-Pin_4): track 5.72 -> 0.00 mm
- net Net-(J4-Pin_4): track 5.39 -> 0.00 mm
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Other:
- board size 140 x 60 mm -> 140 x 65 mm

Commit message: pcb wip
Other:
- board text added: "4 Way Load Cell v0.1"
- board text removed: "Load Cell"
