File: loadcell_4way.kicad_pcb (KiCad board)
At the start: 2 copper layers, 140 x 65 mm, 118 parts, among them J1 USB_B_Micro, J2 Battery, J3 OLDED_Screen, J4 T4145015051-001, J5 T4145015051-001, J6 T4145015051-001, J7 T4145015051-001, Q1 FDS6892A, Q2 BSS138, Q3 SM2331PSA P-MOSFET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

Commit message: pcb wip
Parts:
- moved C32 35.2 mm to (190.6, 80.4), turned to 0 degrees
- moved C16 33.7 mm to (155.4, 80.0)
- moved C19 30.6 mm to (188.8, 82.0)
- moved C34 29.2 mm to (219.4, 83.6), turned to 180 degrees
- moved C31 28.2 mm to (187.0, 80.4), turned to 180 degrees
- moved C15 26.7 mm to (158.8, 80.0)
- moved C33 6.62 mm to (184.4, 86.2), turned to 0 degrees
- moved R17 2.48 mm to (156.2, 84.0), turned to 90 degrees
- moved R29 2.34 mm to (124.8, 84.2), turned to 90 degrees
- moved R28 1.06 mm to (126.6, 84.2), turned to 90 degrees
- moved R18 0.89 mm to (157.8, 84.0), turned to 90 degrees
- moved C18 0.88 mm to (214.6, 86.6)
- moved C12 0.58 mm to (125.4, 86.6)
- moved R19 0.51 mm to (190.0, 84.4)
- moved R20 0.51 mm to (188.0, 84.4)
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Connections:
- C15 pad 1: VDDA -> A2-
- C16 pad 1: A3+ -> A2+
- C16 pad 2: A3- -> GNDA
- C19 pad 1: A4+ -> A3+
- C19 pad 2: A4- -> A3-
- C31 pad 1: A2- -> A3-
- C32 pad 1: A2+ -> A3+
- C33 pad 1: A3- -> VDDA
- C34 pad 1: A3+ -> A4+
- C34 pad 2: GNDA -> A4-
- J4 pad 2: GNDA -> Net-(J4-Pad2)
- J4 pad 3: Net-(J4-Pad3) -> GNDA
- J5 pad 2: GNDA -> Net-(J5-Pad2)
- J5 pad 3: Net-(J5-Pad3) -> GNDA
- J6 pad 2: GNDA -> Net-(J6-Pad2)
- J6 pad 3: Net-(J6-Pad3) -> GNDA
- J7 pad 2: GNDA -> Net-(J7-Pad2)
- J7 pad 3: Net-(J7-Pad3) -> GNDA
- R17 pad 1: Net-(J5-Pad3) -> Net-(J5-Pad4)
- R18 pad 1: Net-(J5-Pad4) -> Net-(J5-Pad2)
- R19 pad 1: Net-(J6-Pad3) -> Net-(J6-Pad4)
- R20 pad 1: Net-(J6-Pad4) -> Net-(J6-Pad2)
- R26 pad 1: Net-(J7-Pad3) -> Net-(J7-Pad4)
- R28 pad 1: Net-(J4-Pad4) -> Net-(J4-Pad2)
- R29 pad 1: Net-(J4-Pad3) -> Net-(J4-Pad4)
- R30 pad 1: Net-(J7-Pad4) -> Net-(J7-Pad2)
Routing:
- net Net-(J4-Pad3): track 9.18 -> 0.00 mm
- net Net-(J6-Pad3): track 8.46 -> 0.00 mm
- net Net-(J7-Pad3): track 7.63 -> 0.00 mm
- net Net-(J5-Pad3): track 7.53 -> 0.00 mm
- net Net-(J4-Pad2): track 0.00 -> 6.29 mm
- net Net-(J5-Pad2): track 0.00 -> 5.27 mm
- net Net-(J6-Pad2): track 0.00 -> 4.60 mm
- net Net-(J7-Pad2): track 0.00 -> 3.52 mm
- net A2+: track 24.6 -> 21.6 mm
- net GNDA: track 4.68 -> 1.81 mm, vias 56 -> 67
- net Net-(J6-Pad4): track 13.5 -> 16.4 mm
- net SHIELD: track 141.3 -> 138.9 mm
- net A1+: track 56.2 -> 54.1 mm
- net Net-(J7-Pad4): track 16.0 -> 14.1 mm
- net VDDA: track 180.0 -> 181.4 mm
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
Commit message: added enclusre fixed lcd spin around and button
Parts:
- moved R14 8.41 mm to (224.4, 69.4)
- moved J3 7.60 mm to (220.0, 61.2), turned to 0 degrees
- moved R16 2.63 mm to (224.4, 66.6)
Connections:
- SW2 pad 1: BTN_3 -> Net-(D4-K)
- SW3 pad 1: Net-(D4-K) -> BTN_3
Routing:
- net Net-(D4-K): track 97.6 -> 39.2 mm, vias 1 -> 3
- net BTN_3: track 78.9 -> 97.8 mm, vias 3 -> 4
- net +3V3: track 227.8 -> 211.3 mm
- net ESP32_IO9: track 143.2 -> 146.1 mm
- net SDA: track 60.9 -> 63.2 mm
- net A4-: track 53.6 -> 52.9 mm
- net A4+: track 54.1 -> 53.4 mm

Commit message: v0.2 wip
Parts:
- removed R38: 10k, Resistor_SMD:R_0603_1608Metric
- removed the SW2 at (134.0, 65.0)
- added FID1: Fiducial, Fiducial:Fiducial_0.5mm_Mask1.5mm, F.Cu at (235.0, 88.5)
- added FID2: Fiducial, Fiducial:Fiducial_0.5mm_Mask1.5mm, F.Cu at (202.5, 48.0)
- added FID3: Fiducial, Fiducial:Fiducial_0.5mm_Mask1.5mm, F.Cu at (106.5, 52.0)
- H1, H2, H3, H4: footprint MountingHole:MountingHole_3.2mm_M3 -> MountingHole:MountingHole_4.3mm_M4
- J2: footprint Connector_JST:JST_PH_B2B-PH-SM4-TB_1x02-1MP_P2.00mm_Vertical -> Loadcell:JST_PH_B2B-PH-SM4-TB_1x02-1MP_P2.00mm_Vertical_long
- moved H1 141.2 mm to (105.0, 40.0)
- moved H2 141.2 mm to (235.0, 40.0)
- moved H3 141.2 mm to (235.0, 95.0)
- moved H4 141.2 mm to (105.0, 95.0)
- moved R33 51.8 mm to (180.6, 65.0), turned to 90 degrees
- moved H5 2.50 mm to (197.5, 78.5)
- moved H6 2.50 mm to (219.5, 56.5)
- moved H7 2.50 mm to (197.5, 56.5)
- moved H8 2.50 mm to (219.5, 78.5)
- moved J1 2.50 mm to (103.5, 67.5)
- moved J3 2.50 mm to (220.0, 63.7)
- moved R16 1.60 mm to (224.4, 68.2)
- moved R14 0.90 mm to (224.4, 70.3)
- moved SW2 0.50 mm to (134.0, 80.5)
- moved J2 0.10 mm to (115.0, 44.9)
- renumbered SW3 to SW2
Connections:
- R33 pad 1: BTN_3 -> +3V3
- R33 pad 2: +3V3 -> PWDN
- SW2 pad 1: BTN_3 -> Net-(D4-K)
- U10 pad 26: Net-(U10-~{PDWN}) -> PWDN
- U4 pad 16: BTN_3 -> PWDN
Routing:
- net BTN_3: track 97.8 -> 0.00 mm, vias 4 -> 0
- net PWDN: track 0.00 -> 31.9 mm
- net Net-(D4-K): track 39.2 -> 56.6 mm
- net +5V: track 115.7 -> 106.0 mm, vias 8 -> 6
- net Net-(U10-~{PDWN}): track 3.85 -> 0.00 mm
- net BAT-: track 25.7 -> 23.1 mm
- net GND: track 46.7 -> 48.8 mm
- net VBUS: track 30.5 -> 32.4 mm
- net +3V3: track 211.3 -> 213.0 mm
- net SDA: track 63.2 -> 64.7 mm
- net D+: track 9.60 -> 10.6 mm
- net D-: track 9.91 -> 10.9 mm
- net A4-: track 52.9 -> 52.4 mm
Other:
- board text added: "4 Way Load Cell v0.2"
- board text removed: "4 Way Load Cell v0.1"

Commit message: v0.2
Parts:
- H1, H2, H3, H4: footprint MountingHole:MountingHole_4.3mm_M4 -> MountingHole:MountingHole_3mm
- Q1: value FDS6892A -> FDS9926A
- moved H2 141.2 mm to (105.0, 95.0)
- moved H4 141.2 mm to (235.0, 40.0)
- moved Q1 0.11 mm to (128.4, 47.0)
