File: loadcell_4way.kicad_sch (KiCad schematic)
At the start: 118 parts, among them J1 USB_B_Micro, J2 Battery, J3 OLDED_Screen, J4 T4145015051-001, J5 T4145015051-001, J6 T4145015051-001, J7 T4145015051-001, Q1 FDS6892A, Q2 BSS138, Q3 SM2331PSA P-MOSFET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

Commit message: v0.2 wip
Parts:
- removed R25: 10k, Resistor_SMD:R_0603_1608Metric, symbol Device:R
- removed SW3: SW_Push, Button_Switch_THT:SW_PUSH_6mm, symbol Switch:SW_Push
- added FID1, FID2, FID3: Fiducial, Fiducial:Fiducial_0.5mm_Mask1.5mm, symbol Mechanical:Fiducial
- H5, H6, H7, H8: footprint MountingHole:MountingHole_3.2mm_M3 -> MountingHole:MountingHole_4.3mm_M4
- J2: footprint Connector_JST:JST_PH_B2B-PH-SM4-TB_1x02-1MP_P2.00mm_Vertical -> Loadcell:JST_PH_B2B-PH-SM4-TB_1x02-1MP_P2.00mm_Vertical_long
Connections:
- net BTN_3 is gone; now on net PWDN: U4.16 (GPIO2/ADC1_CH2)
- net PWDN: now reaches R23.2, U10.26 (~{PDWN})
Other:
- note added: "4way loadcell"
- note added: "v0.2"
- note removed: "Force Gauge"
- note removed: "v0.4"

Commit message: v0.2
Parts:
- removed Q1: FDS6892A, Package_SO:SOIC-8_3.9x4.9mm_P1.27mm, symbol Transistor_FET:FDS6892A
- added Q1: FDS9926A, Package_SO:SOIC-8_3.9x4.9mm_P1.27mm, symbol Transistor_FET:FDS9926A
- H5, H6, H7, H8: footprint MountingHole:MountingHole_4.3mm_M4 -> MountingHole:MountingHole_3mm
Connections:
- net BAT-: now also Q1.3 (S2)
- net GND: now also Q1.1 (S1)
- net at U1.3 (OC): now also Q1.2 (G1)
- new net: Q1.5 (D2), Q1.6 (D2), Q1.7 (D1), Q1.8 (D1)
- new net: Q1.4 (G2), U1.1 (OD)
Changed lines of the file:
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@@
       (effects (font (size 1.27 1.27)) (justify left))
     )
-    (property "Footprint" "MountingHole:MountingHole_4.3mm_M4" (at 135.89 191.77 0)
+    (property "Footprint" "MountingHole:MountingHole_3mm" (at 135.89 191.77 0)
       (effects (font (size 1.27 1.27)) hide)
     )
@@
       (effects (font (size 1.27 1.27)) (justify left))
     )
-    (property "Footprint" "MountingHole:MountingHole_4.3mm_M4" (at 135.89 186.69 0)
+    (property "Footprint" "MountingHole:MountingHole_3mm" (at 135.89 186.69 0)
       (effects (font (size 1.27 1.27)) hide)
     )
@@
     )
   )
+  (symbol (lib_id "Transistor_FET:FDS9926A") (at 39.37 140.97 270) (unit 1)
+    (in_bom yes) (on_board yes) (dnp no) (fields_autoplaced)
+    (property "Reference" "Q1" (at 39.37 147.32 90)
+      (effects (font (size 1.27 1.27)))
+    )
+    (property "Value" "FDS9926A" (at 39.37 149.86 90)
+      (effects (font (size 1.27 1.27)))
+    )
+    (property "Footprint" "Package_SO:SOIC-8_3.9x4.9mm_P1.27mm" (at 37.465 146.05 0)
+      (effects (font (size 1.27 1.27) italic) (justify left) hide)
+    )
+    (property "Datasheet" "https://www.onsemi.com/pub/Collateral/FDS9926A-D.pdf" (at 39.37 140.97 0)
+      (effects (font (size 1.27 1.27)) (justify left) hide)
+    )
+    (pin "1")
+    (pin "2")
+    (pin "7")
+    (pin "8")
+    (pin "3")
+    (pin "4")
+    (pin "5")
+    (pin "6")
+    (instances
+      (project "loadcell_4way"
+        (path "/f1e4dab1-2dd6-4b7a-ae05-4592c2499fb0"
+          (reference "Q1") (unit 1)
+        )
+      )
+    )
+  )
   (symbol (lib_id "Loadcell:T4145015051-001") (at 17.78 318.77 0) (mirror y) (unit 1)
     (in_bom yes) (on_board yes) (dnp no) (fields_autoplaced)
@@
     )
   )
-  (symbol (lib_id "Transistor_FET:FDS6892A") (at 54.61 146.05 90) (unit 2)
-    (in_bom yes) (on_board yes) (dnp no)
-    (property "Reference" "Q1" (at 54.61 137.3632 90)
-      (effects (font (size 1.27 1.27)))
-    )
-    (property "Value" "FDS6892A" (at 54.61 139.6746 90)
-      (effects (font (size 1.27 1.27)))
-    )
-    (property "Footprint" "Package_SO:SOIC-8_3.9x4.9mm_P1.27mm" (at 56.515 140.97 0)
-      (effects (font (size 1.27 1.27) italic) (justify left) hide)
-    )
-    (property "Datasheet" "http://www.fairchildsemi.com/ds/FD/FDS6892A.pdf" (at 54.61 146.05 0)
-      (effects (font (size 1.27 1.27)) (justify left) hide)
-    )
-    (pin "1")
-    (pin "2")
-    (pin "7")
-    (pin "8")
-    (pin "3")
-    (pin "4")
-    (pin "5")
-    (pin "6")
-    (instances
-      (project "forcegauge"
-        (path "/7e1217ba-8a3d-4079-8d7b-b45f90cfbf53"
-          (reference "Q1") (unit 2)
-        )
-      )
-      (project "loadcell_4way"
-        (path "/f1e4dab1-2dd6-4b7a-ae05-4592c2499fb0"
-          (reference "Q1") (unit 2)
-        )
-      )
-    )
-  )
   (symbol (lib_id "power:GNDA") (at 273.05 262.89 0) (unit 1)
     (in_bom yes) (on_board yes) (dnp no) (fields_autoplaced)
@@
     )
   )
+  (symbol (lib_id "Transistor_FET:FDS9926A") (at 54.61 146.05 90) (unit 2)
+    (in_bom yes) (on_board yes) (dnp no) (fields_autoplaced)
+    (property "Reference" "Q1" (at 54.61 137.16 90)
+      (effects (font (size 1.27 1.27)))
+    )
+    (property "Value" "FDS9926A" (at 54.61 139.7 90)
+      (effects (font (size 1.27 1.27)))
+    )
+    (property "Footprint" "Package_SO:SOIC-8_3.9x4.9mm_P1.27mm" (at 56.515 140.97 0)
+      (effects (font (size 1.27 1.27) italic) (justify left) hide)
+    )
+    (property "Datasheet" "https://www.onsemi.com/pub/Collateral/FDS9926A-D.pdf" (at 54.61 146.05 0)
+      (effects (font (size 1.27 1.27)) (justify left) hide)
+    )
+    (pin "1")
+    (pin "2")
+    (pin "7")
+    (pin "8")
+    (pin "3")
+    (pin "4")
+    (pin "5")
+    (pin "6")
+    (instances
+      (project "loadcell_4way"
+        (path "/f1e4dab1-2dd6-4b7a-ae05-4592c2499fb0"
+          (reference "Q1") (unit 2)
+        )
+      )
+    )
+  )
   (symbol (lib_id "Device:C") (at 139.7 303.53 0) (unit 1)
     (in_bom yes) (on_board yes) (dnp no)
@@
       (effects (font (size 1.27 1.27)) (justify left))
     )
-    (property "Footprint" "MountingHole:MountingHole_4.3mm_M4" (at 135.89 181.61 0)
+    (property "Footprint" "MountingHole:MountingHole_3mm" (at 135.89 181.61 0)
       (effects (font (size 1.27 1.27)) hide)
     )
@@
       (effects (font (size 1.27 1.27)) (justify left))
     )
-    (property "Footprint" "MountingHole:MountingHole_4.3mm_M4" (at 135.89 176.53 0)
+    (property "Footprint" "MountingHole:MountingHole_3mm" (at 135.89 176.53 0)
       (effects (font (size 1.27 1.27)) hide)
     )
@@
         )
       )
-    )
-  )
-  (symbol (lib_id "Transistor_FET:FDS6892A") (at 39.37 140.97 270) (unit 1)
-    (in_bom yes) (on_board yes) (dnp no)
-    (property "Reference" "Q1" (at 39.37 147.2946 90)
-      (effects (font (size 1.27 1.27)))
-    )
-    (property "Value" "FDS6892A" (at 39.37 149.606 90)
-      (effects (font (size 1.27 1.27)))
-    )
-    (property "Footprint" "Package_SO:SOIC-8_3.9x4.9mm_P1.27mm" (at 37.465 146.05 0)
-      (effects (font (size 1.27 1.27) italic) (justify left) hide)
-    )
-    (property "Datasheet" "http://www.fairchildsemi.com/ds/FD/FDS6892A.pdf" (at 39.37 140.97 0)
-      (effects (font (size 1.27 1.27)) (justify left) hide)
-    )
-    (property "Alt1" "DMN2041LSD-13" (at 39.37 140.97 90)
-      (effects (font (size 1.27 1.27)) hide)
-    )
-    (property "Alt2" "FDS9926A" (at 39.37 140.97 90)
-      (effects (font (size 1.27 1.27)) hide)
-    )
-    (pin "1")
-    (pin "2")
-    (pin "7")
-    (pin "8")
-    (pin "3")
-    (pin "4")
-    (pin "5")
-    (pin "6")
-    (instances
-      (project "forcegauge"
-        (path "/7e1217ba-8a3d-4079-8d7b-b45f90cfbf53"
-          (reference "Q1") (unit 1)
-        )
-      )
-      (project "loadcell_4way"
-        (path "/f1e4dab1-2dd6-4b7a-ae05-4592c2499fb0"
-          (reference "Q1") (unit 1)
-        )
-      )
